File: schematy_kicad/schema.kicad_sch (KiCad schematic)
At the start: 15 parts, among them J1 MCU_ATmega328P_Module, J2 MCU_ATmega328P_Module, J3 LCD_1602_I2C, J4 MCU_ATmega328P_Module, J5 RF_433MHz_TX, J6 MCU_ATmega328P_Module, J7 RF_433MHz_RX, SW1 BTN_MORSE, SW2 BTN_SPEED_UP, SW3 BTN_SPEED_DOWN

Commit message: Update code ot match MISRA requirements, and add more funcionalities + update kicad schema
Parts:
- added D3: LED_CRNT_SPEED, symbol Device:LED
- added R220Ω: R, symbol Device:R
- added SW4: BTN_CLEAR_LCD, symbol Switch:SW_Push
Connections:
- net GND: now also D3.2 (A), SW4.1
- net at J4.11 (Pin_11): now also SW4.2
- net at J2.11 (Pin_11): now also R220Ω.1
- new net: D3.1 (K), R220Ω.2
Other:
- note added: "D8"
- note added: "Ręczne czyszczenie ekranu"
- note added: "Sygnalizacja aktualnej szybkości interpretacji znaków"
